Commit message: 仿真90度模具可铺

File: src/afp_mjc/env/mujoco_ur5e/ur5e.urdf (robot description, URDF)
Before this commit: robot ur, 11 links, 10 joints
Joints:
- joint flange-tool0: origin xyz=0 0 0.237 rpy=0 0 0 -> xyz=0 0 0.161 rpy=0 0 0

Commit message: 修改urdf

File: src/afp_mjc/env/mujoco_ur5e/ur5e.urdf (robot description, URDF)
Before this commit: robot ur, 11 links, 10 joints
Links:
- link base_link_inertia: geometry collision mesh filename=package://ur_description/meshes/ur5e/collision/base.stl; visual mesh filename=package://ur_description/meshes/ur5e/visual/base.dae
- link forearm_link: mass 2.275 -> 2.846; geometry collision mesh filename=package://ur_description/meshes/ur5e/collision/forearm.stl; visual mesh filename=package://ur_description/meshes/ur5e/visual/forearm.dae
- link shoulder_link: mass 3.7 -> 3.761; geometry collision mesh filename=package://ur_description/meshes/ur5e/collision/shoulder.stl; visual mesh filename=package://ur_description/meshes/ur5e/visual/shoulder.dae
- link upper_arm_link: mass 8.393 -> 8.058; geometry collision mesh filename=package://ur_description/meshes/ur5e/collision/upperarm.stl; visual mesh filename=package://ur_description/meshes/ur5e/visual/upperarm.dae
- link wrist_1_link: mass 1.219 -> 1.37; geometry collision mesh filename=package://ur_description/meshes/ur5e/collision/wrist1.stl; visual mesh filename=package://ur_description/meshes/ur5e/visual/wrist1.dae
- link wrist_2_link: mass 1.219 -> 1.3; geometry collision mesh filename=package://ur_description/meshes/ur5e/collision/wrist2.stl; visual mesh filename=package://ur_description/meshes/ur5e/visual/wrist2.dae
- link wrist_3_link: mass 0.1879 -> 0.365; geometry collision mesh filename=package://ur_description/meshes/ur5e/collision/wrist3.stl; visual mesh filename=package://ur_description/meshes/ur5e/visual/wrist3.dae
Joints:
- joint base_link-base_link_inertia: origin xyz=0 0 0 rpy=0 0 0 -> xyz=0 0 0 rpy=0 0 3.141592653589793
- joint elbow_joint: origin xyz=-0.4255253648975907 0 0 rpy=3.13874389241046 3.137653466693207 3.141586607991614 -> xyz=-0.425 0 0 rpy=0 0 0
- joint flange-tool0: origin xyz=0 0 0.237 rpy=0 0 0 -> xyz=0 0 0.221 rpy=1.5707963267948966 0 1.5707963267948966
- joint shoulder_lift_joint: origin xyz=0.0001081748286041046 0 0 rpy=1.569659240772069 0 6.304982219230273e-06 -> xyz=0 0 0 rpy=1.570796327 0 0
- joint shoulder_pan_joint: origin xyz=0 0 0.1625577379268472 rpy=0 0 -8.69989228782786e-08 -> xyz=0 0 0.1625 rpy=0 0 0
- joint wrist_1_joint: origin xyz=-0.3925097341358023 -0.0005013994603143044 0.133784519987649 rpy=0.003747796178587034 -0.001926900513523302 9.839228519106451e-06 -> xyz=-0.3922 0 0.1333 rpy=0 0 0
- joint wrist_2_joint: origin xyz=0.0001836861607974969 -0.09976037000753009 1.384007358094994e-05 rpy=1.570657593613663 0 3.736438307384589e-06 -> xyz=0 -0.0997 -2.044881182297852e-11 rpy=1.570796327 0 0
- joint wrist_3-flange: origin xyz=0 0 0 rpy=0 0 0 -> xyz=0 0 0 rpy=0 -1.5707963267948966 -1.5707963267948966
- joint wrist_3_joint: origin xyz=-0.0001205608764787091 0.09931578756547574 9.668968792854205e-05 rpy=1.571769884572071 3.141592653589793 3.141592602684103 -> xyz=0 0.0996 -2.042830148012698e-11 rpy=1.570796326589793 3.141592653589793 3.141592653589793

Commit message: urdf tool 0.161->0.221 & 控制器参数微调

File: src/afp_mjc/env/mujoco_ur5e/ur5e.urdf (robot description, URDF)
Before this commit: robot ur, 11 links, 10 joints
Joints:
- joint flange-tool0: origin xyz=0 0 0.161 rpy=0 0 0 -> xyz=0 0 0.221 rpy=0 0 0

Commit message: after pull

File: src/afp_mjc/env/mujoco_ur5e/ur5e.urdf (robot description, URDF)
Before this commit: robot ur5e_robot, 11 links, 10 joints
Links:
- link base_link_inertia: geometry collision mesh filename=/home/lgx/Project/AFP/src/afp_mjc/env/mujoco_ur5e/assets/co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; visual mesh filename=/home/lgx/Project/AFP/src/afp_mjc/env/mujoco_ur5e/assets/vi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
- link forearm_link: mass 2.846 -> 2.275; geometry collision mesh filename=/home/lgx/Project/AFP/src/afp_mjc/env/mujoco_ur5e/assets/co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; visual mesh filename=/home/lgx/Project/AFP/src/afp_mjc/env/mujoco_ur5e/assets/vi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
- link shoulder_link: mass 3.761 -> 3.7; geometry collision mesh filename=/home/lgx/Project/AFP/src/afp_mjc/env/mujoco_ur5e/assets/co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; visual mesh filename=/home/lgx/Project/AFP/src/afp_mjc/env/mujoco_ur5e/assets/vi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
- link upper_arm_link: mass 8.058 -> 8.393; geometry collision mesh filename=/home/lgx/Project/AFP/src/afp_mjc/env/mujoco_ur5e/assets/co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; visual mesh filename=/home/lgx/Project/AFP/src/afp_mjc/env/mujoco_ur5e/assets/vi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
- link wrist_1_link: mass 1.37 -> 1.219; geometry collision mesh filename=/home/lgx/Project/AFP/src/afp_mjc/env/mujoco_ur5e/assets/co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; visual mesh filename=/home/lgx/Project/AFP/src/afp_mjc/env/mujoco_ur5e/assets/vi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
- link wrist_2_link: mass 1.3 -> 1.219; geometry collision mesh filename=/home/lgx/Project/AFP/src/afp_mjc/env/mujoco_ur5e/assets/co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; visual mesh filename=/home/lgx/Project/AFP/src/afp_mjc/env/mujoco_ur5e/assets/vi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
- link wrist_3_link: mass 0.365 -> 0.1879; geometry collision mesh filename=/home/lgx/Project/AFP/src/afp_mjc/env/mujoco_ur5e/assets/co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; visual mesh filename=/home/lgx/Project/AFP/src/afp_mjc/env/mujoco_ur5e/assets/vi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
Joints:
- joint base_link-base_link_inertia: origin xyz=0 0 0 rpy=0 0 3.141592653589793 -> xyz=0 0 0 rpy=0 0 0
- joint elbow_joint: origin xyz=-0.425 0 0 rpy=0 0 0 -> xyz=-0.4255253648975907 0 0 rpy=3.13874389241046 3.137653466693207 3.141586607991614
- joint shoulder_lift_joint: origin xyz=0 0 0 rpy=1.570796327 0 0 -> xyz=0.0001081748286041046 0 0 rpy=1.569659240772069 0 6.304982219230273e-06
- joint shoulder_pan_joint: origin xyz=0 0 0.1625 rpy=0 0 0 -> xyz=0 0 0.1625577379268472 rpy=0 0 -8.69989228782786e-08
- joint wrist_1_joint: origin xyz=-0.3922 0 0.1333 rpy=0 0 0 -> xyz=-0.3925097341358023 -0.0005013994603143044 0.133784519987649 rpy=0.003747796178587034 -0.001926900513523302 9.839228519106451e-06
- joint wrist_2_joint: origin xyz=0 -0.0997 -2.044881182297852e-11 rpy=1.570796327 0 0 -> xyz=0.0001836861607974969 -0.09976037000753009 1.384007358094994e-05 rpy=1.570657593613663 0 3.736438307384589e-06
- joint wrist_3-flange: origin xyz=0 0 0 rpy=0 -1.5707963267948966 -1.5707963267948966 -> xyz=0 0 0 rpy=0 0 0
- joint wrist_3_joint: origin xyz=0 0.0996 -2.042830148012698e-11 rpy=1.570796326589793 3.141592653589793 3.141592653589793 -> xyz=-0.0001205608764787091 0.09931578756547574 9.668968792854205e-05 rpy=1.571769884572071 3.141592653589793 3.141592602684103
